File: 8x8/64panel.sch (EAGLE design)
At the start: 72 parts, among them J1 LED_PADCIRCULARPAD, J2 LED_PADCIRCULARPAD, J3 LED_PADCIRCULARPAD, J4 LED_PADCIRCULARPAD, J5 LED_PADCIRCULARPAD, J6 LED_PADCIRCULARPAD, J7 LED_PADCIRCULARPAD, J8 LED_PADCIRCULARPAD

Commit message: changing to 6-pin
Parts:
- added FRAME1: FRAME-LEDGER, SparkFun-Aesthetics:FRAME-LEDGER
- added LOGO1: SFE_LOGO_NAME_FLAME.2_INCH, SparkFun-Aesthetics:SFE_LOGO_NAME_FLAME.2_INCH
Other:
- moved on the sheet: D1, D10, D11, D12, D13, D14, D15, D16, D17, D18, D19, D2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
